File: Asteroids_PCB/Asteroids_PCB.kicad_pcb (KiCad board)
At the start: 2 copper layers, 290.8 x 482.6 mm, 1469 parts, among them J20 J20, J21 J21, Q1 2N3906, Q10 2N3906, Q11 2N6044, Q12 2N6044, Q13 2N6044, Q14 MPSA06S, Q15 MPSA06S, Q16 2N3906, Q17 2N3906, Q2 2N3906, Q3 2N3906, Q4 2N3906, Q5 2N3906, Q6 2N3643, Q7 2N3906, Q8 2N3904, Q9 2N3904, T1 TPAD1, T10 TPAD, T11 TPAD, T12 TPAD, T13 TPAD, T14 TPAD, T15 TPAD, T16 TPAD, T17 TPAD, T2 TPAD2, T3 TPAD3, T4 TPAD4, T5 TPAD5, T6 TPAD6, T7 TPAD7, U7805 L7805, U7812 L7812, U7815 L7815, U7915 L7915, Y1 12.096MHz

Commit message: Moved the IC silkscreen identifiers to areas they can be seen after soldering
Routing:
- net A11: track 64.9 -> 69.3 mm
Other:
- board text added: "C54"
- board text added: "C55"

Commit message: Changed the silkscreen on the components so the compinent IDs can be seen after soldering
Other:
- board text added: "C9"
- board text added: "Designed By Nick Mikstas"
